File: doc/boards/audio-board/codec.sch (KiCad schematic (older format))
At the start: 30 parts, among them IC13 MK2703B, IC14 CS4272, P3 CONN_01X10, Q3 BC547B, Y1 27M

Commit message: Updated schematics for KiCAD 5
Parts:
- C70, C71, C72, C74, C76, C78, C80, C82, C83, C84: symbol C -> Device:C
- C73, C75, C77, C79, C81: symbol CP -> Device:CP
- IC13: symbol MK2703B -> pedalevite:MK2703B
- IC14: symbol CS4272 -> audio-board-rescue:CS4272
- JP1: symbol Jumper_NC_Dual -> Device:Jumper_NC_Dual
- P3: symbol CONN_01X10 -> conn:CONN_01X10
- Q3: symbol Q_NPN_CBE -> Device:Q_NPN_CBE
- R70, R71, R72, R73: symbol R -> Device:R
- TP1, TP2, TP3, TP4, TP5: symbol TEST -> audio-board-rescue:TEST
- Y1: symbol Crystal -> Device:Crystal
