File: doc/boards/audio-board/connect.sch (KiCad schematic (older format))
At the start: 14 parts, among them P10 IN1SWB, P11 IN2SWB, P14 IN1G, P15 IN2G, P16 OUT1ASYM, P17 OUT2ASYM, P18 OUT1XLR, P19 OUT2XLR, P4 IN1XLR, P5 IN2XLR, P6 IN1TRS, P7 IN2TRS, P8 IN1SWA, P9 IN2SWA

Commit message: Updated schematics for KiCAD 5
Parts:
- P10, P11, P6, P7: symbol CONN_02X03 -> conn:CONN_02X03
- P14, P15, P16, P17, P8, P9: symbol CONN_01X02 -> conn:CONN_01X02
- P18, P19, P4, P5: symbol CONN_01X03 -> conn:CONN_01X03
Changed lines of the file:
@@
-EESchema Schematic File Version 2
-LIBS:power
-LIBS:device
-LIBS:transistors
-LIBS:conn
-LIBS:linear
-LIBS:regul
-LIBS:74xx
-LIBS:cmos4000
-LIBS:adc-dac
-LIBS:memory
-LIBS:xilinx
-LIBS:microcontrollers
-LIBS:dsp
-LIBS:microchip
-LIBS:analog_switches
-LIBS:motorola
-LIBS:texas
-LIBS:intel
-LIBS:audio
-LIBS:interface
-LIBS:digital-audio
-LIBS:philips
-LIBS:display
-LIBS:cypress
-LIBS:siliconi
-LIBS:opto
-LIBS:atmel
-LIBS:contrib
-LIBS:valves
-LIBS:pedalevite
-LIBS:switches
-LIBS:74xgxx
-LIBS:ac-dc
-LIBS:actel
-LIBS:allegro
-LIBS:Altera
-LIBS:analog_devices
-LIBS:battery_management
-LIBS:bbd
-LIBS:brooktre
-LIBS:cmos_ieee
-LIBS:dc-dc
-LIBS:diode
-LIBS:elec-unifil
-LIBS:ESD_Protection
-LIBS:ftdi
-LIBS:gennum
-LIBS:graphic
-LIBS:hc11
-LIBS:ir
-LIBS:Lattice
-LIBS:logo
-LIBS:maxim
-LIBS:mechanical
-LIBS:microchip_dspic33dsc
-LIBS:microchip_pic10mcu
-LIBS:microchip_pic12mcu
-LIBS:microchip_pic16mcu
-LIBS:microchip_pic18mcu
-LIBS:microchip_pic32mcu
-LIBS:motor_drivers
-LIBS:motors
-LIBS:msp430
-LIBS:nordicsemi
-LIBS:nxp_armmcu
-LIBS:onsemi
-LIBS:Oscillators
-LIBS:Power_Management
-LIBS:powerint
-LIBS:pspice
-LIBS:references
-LIBS:relays
-LIBS:rfcom
-LIBS:sensors
-LIBS:silabs
-LIBS:stm8
-LIBS:stm32
-LIBS:supertex
-LIBS:transf
-LIBS:ttl_ieee
-LIBS:video
-LIBS:wiznet
-LIBS:Worldsemi
-LIBS:Xicor
-LIBS:zetex
-LIBS:Zilog
-LIBS:Symbols_DCDC-ACDC-Converter_RevC_20Jul2012
-LIBS:Symbols_EN60617_13Mar2013
-LIBS:Symbols_EN60617-10_HF-Radio_DRAFT_12Sep2013
-LIBS:Symbols_ICs-Diskrete_RevD10
-LIBS:Symbols_ICs-Opto_RevB_16Sep2013
-LIBS:Symbols_Microcontroller_Philips-NXP_RevA_06Oct2013
-LIBS:Symbols_Socket-DIN41612_RevA
-LIBS:Symbols_Transformer-Diskrete_RevA
-LIBS:SymbolsSimilarEN60617+oldDIN617-RevE8
-LIBS:audio-board-cache
-EELAYER 25 0
+EESchema Schematic File Version 4
+EELAYER 30 0
 EELAYER END
 $Descr A4 11693 8268
 encoding utf-8
 Sheet 2 7
-Title "Pédale Vite v2  Audio interface"
+Title "Pédale Vite v2 — Audio interface"
 Date "2019-10-28"
 Rev ""
@@
 $EndDescr
 $Comp
-L CONN_01X02 P17
+L conn:CONN_01X02 P17
 U 1 1 58BC390A
 P 3100 3650
@@
 $EndComp
 $Comp
-L CONN_01X02 P16
+L conn:CONN_01X02 P16
 U 1 1 58BC3904
 P 3000 3650
@@
 $EndComp
 $Comp
-L CONN_01X02 P15
+L conn:CONN_01X02 P15
 U 1 1 58BC3860
 P 4150 2600
@@
 $EndComp
 $Comp
-L CONN_01X02 P14
+L conn:CONN_01X02 P14
 U 1 1 58BC385A
 P 1950 2600
@@
 $EndComp
 $Comp
-L CONN_01X02 P9
+L conn:CONN_01X02 P9
 U 1 1 58BC3745
 P 4200 1250
@@
 $EndComp
 $Comp
-L CONN_01X02 P8
+L conn:CONN_01X02 P8
 U 1 1 58BC36D9
 P 2000 1250
@@
 $EndComp
 $Comp
-L CONN_02X03 P7
+L conn:CONN_02X03 P7
 U 1 1 58BC3653
 P 4150 1700
@@
 $EndComp
 $Comp
-L CONN_02X03 P6
+L conn:CONN_02X03 P6
 U 1 1 58BC34CB
 P 1950 1700
@@
 $EndComp
 $Comp
-L CONN_01X03 P19
+L conn:CONN_01X03 P19
 U 1 1 58BC33F1
 P 3100 4100
@@
 $EndComp
 $Comp
-L CONN_01X03 P18
+L conn:CONN_01X03 P18
 U 1 1 58BC3378
 P 3000 4100
@@
 IN1SWA1
 $Comp
-L CONN_01X03 P5
+L conn:CONN_01X03 P5
 U 1 1 58BC244E
 P 4100 1200
@@
 $EndComp
 $Comp
-L CONN_01X03 P4
+L conn:CONN_01X03 P4
 U 1 1 58BC2330
 P 1900 1200
@@
 IN1XLR2
 $Comp
-L GNDA #PWR01
+L power:GNDA #PWR01
 U 1 1 58D54B66
 P 1000 4700
@@
 Connection ~ 5200 4000
 $Comp
-L CONN_02X03 P10
+L conn:CONN_02X03 P10
 U 1 1 58D651CA
 P 1950 2200
@@
 $EndComp
 $Comp
-L CONN_02X03 P11
+L conn:CONN_02X03 P11
 U 1 1 58D653BE
 P 4150 2200
