File: doc/boards/audio-board/input-1.sch (KiCad schematic (older format))
At the start: 71 parts, among them IC5 INA103, IC6 NE5532, IC7 NE5532, IC8 NE5532

Commit message: Updated schematics for KiCAD 5
Parts:
- C30, C31, C34, C35, C36, C37, C38, C40, C41: symbol CP -> Device:CP
- C32, C33, C39, C42, C43, C44, C45, C46, C47, C48: symbol C -> Device:C
- D10, D11, D12, D13, D18, D19, D20, D21: symbol D_ALT -> Device:D_ALT
- D14, D15, D16, D17: symbol D_Schottky -> Device:D_Schottky
- IC5: symbol INA103 -> pedalevite:INA103
- IC6, IC7, IC8: symbol NE5532 -> linear:NE5532
- L3, L4: symbol L -> Device:L
- R10, R11, R12, R13, R14, R15, R16, R17, R18, R19, R20, R21, R22, R23, R24, R25, R26, R27, R28, R29, R30, R31, R32, R33, R34, R35, R36, R37, R38, R39: symbol R -> Device:R
- TP6, TP7, TP8, TP9: symbol TEST -> audio-board-rescue:TEST
Connections:
- net +15V: now also IC6.8 (V+), IC7.8 (V+), IC8.8 (V+)
- net -15V: now also IC6.4 (V-), IC7.4 (V-), IC8.4 (V-)
Other:
- moved on the sheet: R24, R29
