File: doc/boards/audio-board/input-2.sch (KiCad schematic (older format))
At the start: 71 parts, among them IC10 NE5532, IC11 NE5532, IC12 NE5532, IC9 INA103

Commit message: Updated schematics for KiCAD 5
Parts:
- C50, C51, C54, C55, C56, C57, C58, C60, C61: symbol CP -> Device:CP
- C52, C53, C59, C62, C63, C64, C65, C66, C67, C68: symbol C -> Device:C
- D30, D31, D32, D33, D38, D39, D40, D41: symbol D_ALT -> Device:D_ALT
- D34, D35, D36, D37: symbol D_Schottky -> Device:D_Schottky
- IC10, IC11, IC12: symbol NE5532 -> linear:NE5532
- IC9: symbol INA103 -> pedalevite:INA103
- L5, L6: symbol L -> Device:L
- R40, R41, R42, R43, R44, R45, R46, R47, R48, R49, R50, R51, R52, R53, R54, R55, R56, R57, R58, R59, R60, R61, R62, R63, R64, R65, R66, R67, R68, R69: symbol R -> Device:R
- TP10, TP11, TP12, TP13: symbol TEST -> audio-board-rescue:TEST
Connections:
- net +15V: now also IC10.8 (V+), IC11.8 (V+), IC12.8 (V+)
- net -15V: now also IC10.4 (V-), IC11.4 (V-), IC12.4 (V-)
Other:
- moved on the sheet: R54, R59
