File: doc/boards/audio-board/output.sch (KiCad schematic (older format))
At the start: 44 parts, among them IC15 NE5532, IC16 NE5532, IC17 NE5532

Commit message: Updated schematics for KiCAD 5
Parts:
- C100, C101, C90, C91: symbol CP -> Device:CP
- C102, C103, C104, C105, C92, C93, C94, C95, C96, C97, C98: symbol C -> Device:C
- IC15, IC16, IC17: symbol NE5532 -> linear:NE5532
- R100, R101, R102, R103, R104, R105, R106, R107, R108, R109, R110, R111, R112, R80, R81, R82, R83, R84, R85, R86, R87, R88, R89, R90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: symbol R -> Device:R
