File: doc/boards/audio-board/power-supply.sch (KiCad schematic (older format))
At the start: 31 parts, among them IC3 LM7805CT, IC4 L4931CZ33, P2 CONN_01X03, Q1 BC639, Q2 BC640

Commit message: Updated schematics for KiCAD 5
Parts:
- C10, C12, C13, C16, C17, C18, C21: symbol CP -> Device:CP
- C11, C14, C15, C19, C20, C22, C9: symbol C -> Device:C
- D7, D8: symbol D_ALT -> Device:D_ALT
- D9: symbol TL431LP -> references:TL431LP
- IC3: symbol LM7805CT -> regul:LM7805CT
- IC4: symbol L4931CZ33 -> pedalevite:L4931CZ33
- JP2: symbol Jumper_NO_Small -> Device:Jumper_NO_Small
- L7: symbol Ferrite_Bead -> Device:Ferrite_Bead
- P2: symbol CONN_01X03 -> conn:CONN_01X03
- Q1: symbol Q_NPN_ECB -> Device:Q_NPN_ECB
- Q2: symbol Q_PNP_ECB -> Device:Q_PNP_ECB
- R3, R4, R5, R6, R7, R8, R9: symbol R -> Device:R
