File: doc/boards/main-board/main-board.sch (KiCad schematic (older format))
At the start: 117 parts, among them P1 Raspberry_Pi_2_3, P10 ROTENC 7 SW, P11 ROTENC 1, P12 ROTENC 2, P13 ROTENC 3, P14 ROTENC 4, P15 ROTENC 5, P16 DISPLAY, P2 FOOTSW, P3 NAV SW, P4 AUDIO BOARD, P5 LEDS, P6 EXPR 0, P7 EXPR 1, P8 EXPR 2, P9 ROTENC 6 SW, Q1 BC547, Q2 BC547, Q3 BC547, U1 MCP3008, U3 MCP23017, U4 MCP23017

Commit message: Updated schematics for KiCAD 5
Parts:
- C1, C2, C26, C3, C4, C5, C7: symbol C -> Device:C
- C10, C11, C12, C13, C14, C15, C16, C17, C18, C19, C20, C21, C22, C23, C24, C25, C27, C28, C29, C30, C31, C32, C33, C34, C35, C36, C37, C38, C39, C40, C41, C42, C8, C9: symbol C_Small -> Device:C_Small
- MK1, MK2, MK3, MK4: symbol Mounting_Hole -> main-board-rescue:Mounting_Hole
- P1: symbol Raspberry_Pi_2_3 -> conn:Raspberry_Pi_2_3
- P10, P5, P9: symbol CONN_01X04 -> conn:CONN_01X04
- P11, P12, P13, P14, P15, P6, P7, P8: symbol CONN_01X03 -> conn:CONN_01X03
- P16, P3: symbol CONN_02X04 -> conn:CONN_02X04
- P2: symbol CONN_02X08 -> conn:CONN_02X08
- P4: symbol CONN_01X10 -> conn:CONN_01X10
- Q1, Q2, Q3: symbol BC547 -> transistors:BC547
- R1, R2, R3, R4, R5, R6, R7, R77, R78, R79: symbol R -> Device:R
- R26, R27, R28, R29, R30, R31, R32, R33, R34, R35, R36, R37, R38, R39, R40, R41, R42, R43, R60, R61, R62, R63, R64, R65, R66, R67, R68, R69, R70, R71, R72, R73, R74, R75, R8, R9: symbol R_Small -> Device:R_Small
- RN10-17, RN18-25, RN44-51, RN52-59: symbol R_Network08 -> Device:R_Network08
- U1: symbol MCP3008x -> pedalevite:MCP3008x
- U3, U4: symbol MCP23017 -> microchip:MCP23017
