File: doc/boards/misc-boards/but-nav.sch (KiCad schematic (older format))
At the start: 11 parts, among them P400 NAV SW, SW400 SELECT, SW401 ESCAPE, SW402 UP, SW403 DOWN, SW404 LEFT, SW405 RIGHT

Commit message: Updated schematics for KiCAD 5
Parts:
- MK401, MK402, MK403, MK404: symbol Mounting_Hole -> misc-boards-rescue:Mounting_Hole
- P400: symbol CONN_02X04 -> conn:CONN_02X04
- SW400, SW401, SW402, SW403, SW404, SW405: symbol SW_Push -> switches:SW_Push
Changed lines of the file:
@@
-EESchema Schematic File Version 2
-LIBS:power
-LIBS:device
-LIBS:transistors
-LIBS:conn
-LIBS:linear
-LIBS:regul
-LIBS:74xx
-LIBS:cmos4000
-LIBS:adc-dac
-LIBS:memory
-LIBS:xilinx
-LIBS:microcontrollers
-LIBS:dsp
-LIBS:microchip
-LIBS:analog_switches
-LIBS:motorola
-LIBS:texas
-LIBS:intel
-LIBS:audio
-LIBS:interface
-LIBS:digital-audio
-LIBS:philips
-LIBS:display
-LIBS:cypress
-LIBS:siliconi
-LIBS:opto
-LIBS:atmel
-LIBS:contrib
-LIBS:valves
-LIBS:pedalevite
-LIBS:74xgxx
-LIBS:ac-dc
-LIBS:actel
-LIBS:allegro
-LIBS:Altera
-LIBS:analog_devices
-LIBS:battery_management
-LIBS:bbd
-LIBS:bosch
-LIBS:brooktre
-LIBS:cmos_ieee
-LIBS:dc-dc
-LIBS:diode
-LIBS:elec-unifil
-LIBS:ESD_Protection
-LIBS:ftdi
-LIBS:gennum
-LIBS:graphic
-LIBS:hc11
-LIBS:ir
-LIBS:Lattice
-LIBS:leds
-LIBS:logo
-LIBS:maxim
-LIBS:mechanical
-LIBS:microchip_dspic33dsc
-LIBS:microchip_pic10mcu
-LIBS:microchip_pic12mcu
-LIBS:microchip_pic16mcu
-LIBS:microchip_pic18mcu
-LIBS:microchip_pic24mcu
-LIBS:microchip_pic32mcu
-LIBS:modules
-LIBS:motor_drivers
-LIBS:motors
-LIBS:msp430
-LIBS:nordicsemi
-LIBS:nxp
-LIBS:nxp_armmcu
-LIBS:onsemi
-LIBS:Oscillators
-LIBS:Power_Management
-LIBS:powerint
-LIBS:pspice
-LIBS:references
-LIBS:relays
-LIBS:rfcom
-LIBS:sensors
-LIBS:silabs
-LIBS:stm8
-LIBS:stm32
-LIBS:supertex
-LIBS:switches
-LIBS:transf
-LIBS:triac_thyristor
-LIBS:ttl_ieee
-LIBS:video
-LIBS:wiznet
-LIBS:Worldsemi
-LIBS:Xicor
-LIBS:zetex
-LIBS:Zilog
-LIBS:misc-boards-cache
-EELAYER 25 0
+EESchema Schematic File Version 4
+EELAYER 30 0
 EELAYER END
 $Descr A4 11693 8268
@@
 $EndDescr
 $Comp
-L CONN_02X04 P400
+L conn:CONN_02X04 P400
 U 1 1 5D8AB70B
 P 4450 3050
@@
 1, 2: GND, 3: Select, 5: Escape,\n4: Up, 6: Down, 8: Left, 7: Right
 $Comp
-L SW_Push SW402
+L switches:SW_Push SW402
 U 1 1 5D8B4871
 P 5300 3000
@@
 $EndComp
 $Comp
-L SW_Push SW403
+L switches:SW_Push SW403
 U 1 1 5D8B491C
 P 5300 3300
@@
 $EndComp
 $Comp
-L SW_Push SW404
+L switches:SW_Push SW404
 U 1 1 5D8B4945
 P 5300 3600
@@
 $EndComp
 $Comp
-L SW_Push SW400
+L switches:SW_Push SW400
 U 1 1 5D8B4971
 P 3600 3000
@@
 $EndComp
 $Comp
-L SW_Push SW401
+L switches:SW_Push SW401
 U 1 1 5D8B4A24
 P 3600 3300
@@
 $EndComp
 $Comp
-L SW_Push SW405
+L switches:SW_Push SW405
 U 1 1 5D8B4A52
 P 3600 3600
@@
 Connection ~ 3300 3300
 $Comp
-L Mounting_Hole MK401
+L misc-boards-rescue:Mounting_Hole MK401
 U 1 1 5D8D2963
 P 6600 2900
+AR Path="/5D8D2963" Ref="MK401"  Part="1"
+AR Path="/5D8A11C9/5D8D2963" Ref="MK401"  Part="1"
 F 0 "MK401" H 6600 3100 50  0000 C CNN
 F 1 "Mounting_Hole" H 6600 3025 50  0000 C CNN
@@
 $EndComp
 $Comp
-L Mounting_Hole MK402
+L misc-boards-rescue:Mounting_Hole MK402
 U 1 1 5D8D296A
 P 7200 2900
+AR Path="/5D8D296A" Ref="MK402"  Part="1"
+AR Path="/5D8A11C9/5D8D296A" Ref="MK402"  Part="1"
 F 0 "MK402" H 7200 3100 50  0000 C CNN
 F 1 "Mounting_Hole" H 7200 3025 50  0000 C CNN
@@
 $EndComp
 $Comp
-L Mounting_Hole MK403
+L misc-boards-rescue:Mounting_Hole MK403
 U 1 1 5D8D2971
 P 6600 3300
+AR Path="/5D8D2971" Ref="MK403"  Part="1"
+AR Path="/5D8A11C9/5D8D2971" Ref="MK403"  Part="1"
 F 0 "MK403" H 6600 3500 50  0000 C CNN
 F 1 "Mounting_Hole" H 6600 3425 50  0000 C CNN
@@
 $EndComp
 $Comp
-L Mounting_Hole MK404
+L misc-boards-rescue:Mounting_Hole MK404
 U 1 1 5D8D2978
 P 7200 3300
+AR Path="/5D8D2978" Ref="MK404"  Part="1"
+AR Path="/5D8A11C9/5D8D2978" Ref="MK404"  Part="1"
 F 0 "MK404" H 7200 3500 50  0000 C CNN
 F 1 "Mounting_Hole" H 7200 3425 50  0000 C CNN
