File: doc/boards/misc-boards/leds.sch (KiCad schematic (older format))
At the start: 6 parts, among them P100 LEDS

Commit message: Updated schematics for KiCAD 5
Parts:
- D100, D101, D102: symbol LED_ALT -> Device:LED_ALT
- MK101, MK102: symbol Mounting_Hole -> misc-boards-rescue:Mounting_Hole
- P100: symbol CONN_01X04 -> conn:CONN_01X04
Changed lines of the file:
@@
-EESchema Schematic File Version 2
-LIBS:power
-LIBS:device
-LIBS:transistors
-LIBS:conn
-LIBS:linear
-LIBS:regul
-LIBS:74xx
-LIBS:cmos4000
-LIBS:adc-dac
-LIBS:memory
-LIBS:xilinx
-LIBS:microcontrollers
-LIBS:dsp
-LIBS:microchip
-LIBS:analog_switches
-LIBS:motorola
-LIBS:texas
-LIBS:intel
-LIBS:audio
-LIBS:interface
-LIBS:digital-audio
-LIBS:philips
-LIBS:display
-LIBS:cypress
-LIBS:siliconi
-LIBS:opto
-LIBS:atmel
-LIBS:contrib
-LIBS:valves
-LIBS:pedalevite
-LIBS:74xgxx
-LIBS:ac-dc
-LIBS:actel
-LIBS:allegro
-LIBS:Altera
-LIBS:analog_devices
-LIBS:battery_management
-LIBS:bbd
-LIBS:bosch
-LIBS:brooktre
-LIBS:cmos_ieee
-LIBS:dc-dc
-LIBS:diode
-LIBS:elec-unifil
-LIBS:ESD_Protection
-LIBS:ftdi
-LIBS:gennum
-LIBS:graphic
-LIBS:hc11
-LIBS:ir
-LIBS:Lattice
-LIBS:leds
-LIBS:logo
-LIBS:maxim
-LIBS:mechanical
-LIBS:microchip_dspic33dsc
-LIBS:microchip_pic10mcu
-LIBS:microchip_pic12mcu
-LIBS:microchip_pic16mcu
-LIBS:microchip_pic18mcu
-LIBS:microchip_pic24mcu
-LIBS:microchip_pic32mcu
-LIBS:modules
-LIBS:motor_drivers
-LIBS:motors
-LIBS:msp430
-LIBS:nordicsemi
-LIBS:nxp
-LIBS:nxp_armmcu
-LIBS:onsemi
-LIBS:Oscillators
-LIBS:Power_Management
-LIBS:powerint
-LIBS:pspice
-LIBS:references
-LIBS:relays
-LIBS:rfcom
-LIBS:sensors
-LIBS:silabs
-LIBS:stm8
-LIBS:stm32
-LIBS:supertex
-LIBS:switches
-LIBS:transf
-LIBS:triac_thyristor
-LIBS:ttl_ieee
-LIBS:video
-LIBS:wiznet
-LIBS:Worldsemi
-LIBS:Xicor
-LIBS:zetex
-LIBS:Zilog
-LIBS:misc-boards-cache
-EELAYER 25 0
+EESchema Schematic File Version 4
+EELAYER 30 0
 EELAYER END
 $Descr A4 11693 8268
@@
 $EndDescr
 $Comp
-L LED_ALT D100
+L Device:LED_ALT D100
 U 1 1 5D8A5BF4
 P 4450 1400
@@
 $EndComp
 $Comp
-L LED_ALT D101
+L Device:LED_ALT D101
 U 1 1 5D8A5C38
 P 4450 1800
@@
 $EndComp
 $Comp
-L LED_ALT D102
+L Device:LED_ALT D102
 U 1 1 5D8A5C5A
 P 4450 2200
@@
 $EndComp
 $Comp
-L CONN_01X04 P100
+L conn:CONN_01X04 P100
 U 1 1 5D8A6868
 P 5500 1550
@@
 	4800 1500 5300 1500
 $Comp
-L Mounting_Hole MK101
+L misc-boards-rescue:Mounting_Hole MK101
 U 1 1 5D8D304D
 P 6300 1700
+AR Path="/5D8D304D" Ref="MK101"  Part="1"
+AR Path="/5D89DA36/5D8D304D" Ref="MK101"  Part="1"
 F 0 "MK101" H 6300 1900 50  0000 C CNN
 F 1 "Mounting_Hole" H 6300 1825 50  0000 C CNN
@@
 $EndComp
 $Comp
-L Mounting_Hole MK102
+L misc-boards-rescue:Mounting_Hole MK102
 U 1 1 5D8D3054
 P 6900 1700
+AR Path="/5D8D3054" Ref="MK102"  Part="1"
+AR Path="/5D89DA36/5D8D3054" Ref="MK102"  Part="1"
 F 0 "MK102" H 6900 1900 50  0000 C CNN
 F 1 "Mounting_Hole" H 6900 1825 50  0000 C CNN
