File: doc/boards/misc-boards/psu.sch (KiCad schematic (older format))
At the start: 6 parts, among them J501 230VAC, J502 5VDC, U501 RAC15-05SK

Commit message: Updated schematics for KiCAD 5
Parts:
- J501, J502: symbol CONN_01X02 -> conn:CONN_01X02
- MK501, MK502, MK503: symbol Mounting_Hole -> misc-boards-rescue:Mounting_Hole
- U501: symbol IRM-02-5 -> ac-dc:IRM-02-5
Changed lines of the file:
@@
-EESchema Schematic File Version 2
-LIBS:power
-LIBS:device
-LIBS:transistors
-LIBS:conn
-LIBS:linear
-LIBS:regul
-LIBS:74xx
-LIBS:cmos4000
-LIBS:adc-dac
-LIBS:memory
-LIBS:xilinx
-LIBS:microcontrollers
-LIBS:dsp
-LIBS:microchip
-LIBS:analog_switches
-LIBS:motorola
-LIBS:texas
-LIBS:intel
-LIBS:audio
-LIBS:interface
-LIBS:digital-audio
-LIBS:philips
-LIBS:display
-LIBS:cypress
-LIBS:siliconi
-LIBS:opto
-LIBS:atmel
-LIBS:contrib
-LIBS:valves
-LIBS:pedalevite
-LIBS:74xgxx
-LIBS:ac-dc
-LIBS:actel
-LIBS:allegro
-LIBS:Altera
-LIBS:analog_devices
-LIBS:battery_management
-LIBS:bbd
-LIBS:bosch
-LIBS:brooktre
-LIBS:cmos_ieee
-LIBS:dc-dc
-LIBS:diode
-LIBS:elec-unifil
-LIBS:ESD_Protection
-LIBS:ftdi
-LIBS:gennum
-LIBS:graphic
-LIBS:hc11
-LIBS:ir
-LIBS:Lattice
-LIBS:leds
-LIBS:logo
-LIBS:maxim
-LIBS:mechanical
-LIBS:microchip_dspic33dsc
-LIBS:microchip_pic10mcu
-LIBS:microchip_pic12mcu
-LIBS:microchip_pic16mcu
-LIBS:microchip_pic18mcu
-LIBS:microchip_pic24mcu
-LIBS:microchip_pic32mcu
-LIBS:modules
-LIBS:motor_drivers
-LIBS:motors
-LIBS:msp430
-LIBS:nordicsemi
-LIBS:nxp
-LIBS:nxp_armmcu
-LIBS:onsemi
-LIBS:Oscillators
-LIBS:Power_Management
-LIBS:powerint
-LIBS:pspice
-LIBS:references
-LIBS:relays
-LIBS:rfcom
-LIBS:sensors
-LIBS:silabs
-LIBS:stm8
-LIBS:stm32
-LIBS:supertex
-LIBS:switches
-LIBS:transf
-LIBS:triac_thyristor
-LIBS:ttl_ieee
-LIBS:video
-LIBS:wiznet
-LIBS:Worldsemi
-LIBS:Xicor
-LIBS:zetex
-LIBS:Zilog
-LIBS:misc-boards-cache
-EELAYER 25 0
+EESchema Schematic File Version 4
+EELAYER 30 0
 EELAYER END
 $Descr A4 11693 8268
@@
 $EndDescr
 $Comp
-L IRM-02-5 U501
+L ac-dc:IRM-02-5 U501
 U 1 1 5D924859
 P 5100 3600
@@
 	5900 3600 6000 3600
 $Comp
-L CONN_01X02 J502
+L conn:CONN_01X02 J502
 U 1 1 5D920686
 P 6200 3550
@@
 $EndComp
 $Comp
-L CONN_01X02 J501
+L conn:CONN_01X02 J501
 U 1 1 5D9206F7
 P 4700 3550
@@
 $EndComp
 $Comp
-L PWR_FLAG #FLG01
+L power:PWR_FLAG #FLG01
 U 1 1 5D920A47
 P 5000 3300
@@
 $EndComp
 $Comp
-L PWR_FLAG #FLG02
+L power:PWR_FLAG #FLG02
 U 1 1 5D920A6B
 P 5000 3800
@@
 Connection ~ 5000 3500
 $Comp
-L Mounting_Hole MK501
+L misc-boards-rescue:Mounting_Hole MK501
 U 1 1 5D9223FA
 P 7100 3400
+AR Path="/5D9223FA" Ref="MK501"  Part="1"
+AR Path="/5D9245F3/5D9223FA" Ref="MK501"  Part="1"
 F 0 "MK501" H 7100 3600 50  0000 C CNN
 F 1 "Mounting_Hole" H 7100 3525 50  0000 C CNN
@@
 $EndComp
 $Comp
-L Mounting_Hole MK502
+L misc-boards-rescue:Mounting_Hole MK502
 U 1 1 5D922408
 P 7100 3800
+AR Path="/5D922408" Ref="MK502"  Part="1"
+AR Path="/5D9245F3/5D922408" Ref="MK502"  Part="1"
 F 0 "MK502" H 7100 4000 50  0000 C CNN
 F 1 "Mounting_Hole" H 7100 3925 50  0000 C CNN
@@
 $EndComp
 $Comp
-L Mounting_Hole MK503
+L misc-boards-rescue:Mounting_Hole MK503
 U 1 1 5D92240F
 P 7700 3800
+AR Path="/5D92240F" Ref="MK503"  Part="1"
+AR Path="/5D9245F3/5D92240F" Ref="MK503"  Part="1"
 F 0 "MK503" H 7700 4000 50  0000 C CNN
 F 1 "Mounting_Hole" H 7700 3925 50  0000 C CNN
