File: doc/boards/misc-boards/rot-enc-nav.sch (KiCad schematic (older format))
At the start: 4 parts, among them P300 ROTENC 6 SW, P301 ROTENC 7 SW, SW300 UP-DOWN, SW301 LEFT-RIGHT

Commit message: Updated schematics for KiCAD 5
Parts:
- P300, P301: symbol CONN_01X04 -> conn:CONN_01X04
- SW300, SW301: symbol Rotary_Encoder_Switch -> misc-boards-rescue:Rotary_Encoder_Switch
Changed lines of the file:
@@
-EESchema Schematic File Version 2
-LIBS:power
-LIBS:device
-LIBS:transistors
-LIBS:conn
-LIBS:linear
-LIBS:regul
-LIBS:74xx
-LIBS:cmos4000
-LIBS:adc-dac
-LIBS:memory
-LIBS:xilinx
-LIBS:microcontrollers
-LIBS:dsp
-LIBS:microchip
-LIBS:analog_switches
-LIBS:motorola
-LIBS:texas
-LIBS:intel
-LIBS:audio
-LIBS:interface
-LIBS:digital-audio
-LIBS:philips
-LIBS:display
-LIBS:cypress
-LIBS:siliconi
-LIBS:opto
-LIBS:atmel
-LIBS:contrib
-LIBS:valves
-LIBS:pedalevite
-LIBS:74xgxx
-LIBS:ac-dc
-LIBS:actel
-LIBS:allegro
-LIBS:Altera
-LIBS:analog_devices
-LIBS:battery_management
-LIBS:bbd
-LIBS:bosch
-LIBS:brooktre
-LIBS:cmos_ieee
-LIBS:dc-dc
-LIBS:diode
-LIBS:elec-unifil
-LIBS:ESD_Protection
-LIBS:ftdi
-LIBS:gennum
-LIBS:graphic
-LIBS:hc11
-LIBS:ir
-LIBS:Lattice
-LIBS:leds
-LIBS:logo
-LIBS:maxim
-LIBS:mechanical
-LIBS:microchip_dspic33dsc
-LIBS:microchip_pic10mcu
-LIBS:microchip_pic12mcu
-LIBS:microchip_pic16mcu
-LIBS:microchip_pic18mcu
-LIBS:microchip_pic24mcu
-LIBS:microchip_pic32mcu
-LIBS:modules
-LIBS:motor_drivers
-LIBS:motors
-LIBS:msp430
-LIBS:nordicsemi
-LIBS:nxp
-LIBS:nxp_armmcu
-LIBS:onsemi
-LIBS:Oscillators
-LIBS:Power_Management
-LIBS:powerint
-LIBS:pspice
-LIBS:references
-LIBS:relays
-LIBS:rfcom
-LIBS:sensors
-LIBS:silabs
-LIBS:stm8
-LIBS:stm32
-LIBS:supertex
-LIBS:switches
-LIBS:transf
-LIBS:triac_thyristor
-LIBS:ttl_ieee
-LIBS:video
-LIBS:wiznet
-LIBS:Worldsemi
-LIBS:Xicor
-LIBS:zetex
-LIBS:Zilog
-LIBS:misc-boards-cache
-EELAYER 25 0
+EESchema Schematic File Version 4
+EELAYER 30 0
 EELAYER END
 $Descr A4 11693 8268
@@
 $EndDescr
 $Comp
-L CONN_01X04 P301
+L conn:CONN_01X04 P301
 U 1 1 5D8A84AF
 P 4300 2950
@@
 $EndComp
 $Comp
-L CONN_01X04 P300
+L conn:CONN_01X04 P300
 U 1 1 5D8A84B6
 P 4300 1950
@@
 $EndComp
 $Comp
-L Rotary_Encoder_Switch SW300
+L misc-boards-rescue:Rotary_Encoder_Switch SW300
 U 1 1 5D8AE547
 P 5300 1900
@@
 $EndComp
 $Comp
-L Rotary_Encoder_Switch SW301
+L misc-boards-rescue:Rotary_Encoder_Switch SW301
 U 1 1 5D8AE58D
 P 5300 2900
