File: doc/boards/misc-boards/rot-enc-param.sch (KiCad schematic (older format))
At the start: 10 parts, among them P200 ROTENC 1, P201 ROTENC 2, P202 ROTENC 3, P203 ROTENC 4, P204 ROTENC 5, SW200 PARAM 0, SW201 PARAM 1, SW202 PARAM 2, SW203 PARAM 3, SW204 PARAM 4

Commit message: Updated schematics for KiCAD 5
Parts:
- P200, P201, P202, P203, P204: symbol CONN_01X03 -> conn:CONN_01X03
- SW200, SW201, SW202, SW203, SW204: symbol Rotary_Encoder_Switch -> misc-boards-rescue:Rotary_Encoder_Switch
Changed lines of the file:
@@
-EESchema Schematic File Version 2
-LIBS:power
-LIBS:device
-LIBS:transistors
-LIBS:conn
-LIBS:linear
-LIBS:regul
-LIBS:74xx
-LIBS:cmos4000
-LIBS:adc-dac
-LIBS:memory
-LIBS:xilinx
-LIBS:microcontrollers
-LIBS:dsp
-LIBS:microchip
-LIBS:analog_switches
-LIBS:motorola
-LIBS:texas
-LIBS:intel
-LIBS:audio
-LIBS:interface
-LIBS:digital-audio
-LIBS:philips
-LIBS:display
-LIBS:cypress
-LIBS:siliconi
-LIBS:opto
-LIBS:atmel
-LIBS:contrib
-LIBS:valves
-LIBS:pedalevite
-LIBS:74xgxx
-LIBS:ac-dc
-LIBS:actel
-LIBS:allegro
-LIBS:Altera
-LIBS:analog_devices
-LIBS:battery_management
-LIBS:bbd
-LIBS:bosch
-LIBS:brooktre
-LIBS:cmos_ieee
-LIBS:dc-dc
-LIBS:diode
-LIBS:elec-unifil
-LIBS:ESD_Protection
-LIBS:ftdi
-LIBS:gennum
-LIBS:graphic
-LIBS:hc11
-LIBS:ir
-LIBS:Lattice
-LIBS:leds
-LIBS:logo
-LIBS:maxim
-LIBS:mechanical
-LIBS:microchip_dspic33dsc
-LIBS:microchip_pic10mcu
-LIBS:microchip_pic12mcu
-LIBS:microchip_pic16mcu
-LIBS:microchip_pic18mcu
-LIBS:microchip_pic24mcu
-LIBS:microchip_pic32mcu
-LIBS:modules
-LIBS:motor_drivers
-LIBS:motors
-LIBS:msp430
-LIBS:nordicsemi
-LIBS:nxp
-LIBS:nxp_armmcu
-LIBS:onsemi
-LIBS:Oscillators
-LIBS:Power_Management
-LIBS:powerint
-LIBS:pspice
-LIBS:references
-LIBS:relays
-LIBS:rfcom
-LIBS:sensors
-LIBS:silabs
-LIBS:stm8
-LIBS:stm32
-LIBS:supertex
-LIBS:switches
-LIBS:transf
-LIBS:triac_thyristor
-LIBS:ttl_ieee
-LIBS:video
-LIBS:wiznet
-LIBS:Worldsemi
-LIBS:Xicor
-LIBS:zetex
-LIBS:Zilog
-LIBS:misc-boards-cache
-EELAYER 25 0
+EESchema Schematic File Version 4
+EELAYER 30 0
 EELAYER END
 $Descr A4 11693 8268
@@
 $EndDescr
 $Comp
-L CONN_01X03 P204
+L conn:CONN_01X03 P204
 U 1 1 5D8A82DA
 P 4000 5600
@@
 $EndComp
 $Comp
-L CONN_01X03 P200
+L conn:CONN_01X03 P200
 U 1 1 5D8A82E1
 P 4000 2800
@@
 $EndComp
 $Comp
-L CONN_01X03 P201
+L conn:CONN_01X03 P201
 U 1 1 5D8A82E8
 P 4000 3500
@@
 $EndComp
 $Comp
-L CONN_01X03 P202
+L conn:CONN_01X03 P202
 U 1 1 5D8A82EF
 P 4000 4200
@@
 $EndComp
 $Comp
-L CONN_01X03 P203
+L conn:CONN_01X03 P203
 U 1 1 5D8A82F6
 P 4000 4900
@@
 	5300 5700 4200 5700
 $Comp
-L Rotary_Encoder_Switch SW200
+L misc-boards-rescue:Rotary_Encoder_Switch SW200
 U 1 1 5D8B5CF1
 P 5600 2800
@@
 $EndComp
 $Comp
-L Rotary_Encoder_Switch SW201
+L misc-boards-rescue:Rotary_Encoder_Switch SW201
 U 1 1 5D8B5E2F
 P 5600 3500
@@
 $EndComp
 $Comp
-L Rotary_Encoder_Switch SW202
+L misc-boards-rescue:Rotary_Encoder_Switch SW202
 U 1 1 5D8B5E6E
 P 5600 4200
@@
 $EndComp
 $Comp
-L Rotary_Encoder_Switch SW203
+L misc-boards-rescue:Rotary_Encoder_Switch SW203
 U 1 1 5D8B5EAE
 P 5600 4900
@@
 $EndComp
 $Comp
-L Rotary_Encoder_Switch SW204
+L misc-boards-rescue:Rotary_Encoder_Switch SW204
 U 1 1 5D8B5EF0
 P 5600 5600
