File: doc/boards/misc-boards/misc-boards.kicad_pcb (KiCad board)
At the start: 2 copper layers, 210.8 x 160 mm, 37 parts, among them J501 230VAC, J502 5VDC, P100 LEDS, P200 ROTENC 1, P201 ROTENC 2, P202 ROTENC 3, P203 ROTENC 4, P204 ROTENC 5, P300 ROTENC 6 SW, P301 ROTENC 7 SW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

Commit message: Updated board files to KiCAD 6
Other:
- net class Default removed
- net class Power removed
