File: doc/boards/psu-2x15v-ac-dc/psu-2x15v-ac-dc.sch (KiCad schematic (older format))
At the start: 22 parts, among them IC1 LM7815CT, IC2 LM7915CT, J7 Screw_Terminal_1x02, J9 Screw_Terminal_1x02, P1 CONN_01X03, P20 CONN_02X02

Commit message: Updated schematics for KiCAD 5
Parts:
- C1, C2, C5, C6: symbol CP -> Device:CP
- C3, C4, C7, C8: symbol C -> Device:C
- D1, D2, D3, D4, D5, D6: symbol D_ALT -> Device:D_ALT
- IC1: symbol LM7815CT -> regul:LM7815CT
- IC2: symbol LM7915CT -> regul:LM7915CT
- J7, J9: symbol Screw_Terminal_1x02 -> conn:Screw_Terminal_1x02
- L1, L2: symbol L -> Device:L
- P1: symbol CONN_01X03 -> conn:CONN_01X03
- P20: symbol CONN_02X02 -> conn:CONN_02X02
